File: i2c.kicad_sch (KiCad schematic)
At the start: 0 parts

Commit message: added emmc and sd
Parts:
- added U4: MB85RC1MTPNF-G-JNERE1, MB85RC1MTPNF-G-JNERE1:SOIC127P600X175-8N, symbol SamacSys_Parts:MB85RC1MTPNF-G-JNERE1
Connections:
- net I2C_SCL_BUS: now also U4.6 (SCL)
- net I2C_SDA_BUS: now also U4.5 (SDA)
- new net +3.3V: U4.8 (VDD)
- new net FRAM_WP: U4.7 (WP)
- new net GND: U4.2 (A1), U4.3 (A2), U4.4 (VSS)
