File: osd3358 b c.kicad_sch (KiCad schematic)
At the start: 11 parts, among them U1 OSD3358-512M-ISM, Y1 ABM8AIG-24.000MHZ-12-2Z-T3, Y2 ABS07-32.768KHZ-T

Commit message: added emmc and sd
Parts:
- added C17: 2.2uF, symbol Device:C
- added C18: 10uF, symbol Device:C_Small
- added C19, C20, C21, C22: 0.1uF, symbol Device:C_Small
- added IC2: SDINBDA4-32G, BGA153C50P14X14_1150X1300X100, symbol SamacSys_Parts:SDINBDA4-32G
- added J3: Micro_SD_Card, symbol Connector:Micro_SD_Card
- added RN1: 10k, symbol Device:R_Pack11
- added RN2: R_Pack06, symbol Device:R_Pack06
Connections:
- net GND: now also C17.2, C18.2, C19.2, C20.2, C21.2, C22.2, IC2.A6 (VSS_1), IC2.C4 (VSSQ_1), IC2.E7 (VSS_2), IC2.G5 (VSS_3), IC2.H10 (VSS_4), IC2.J5 (VSS_5), IC2.K8 (VSS_6), IC2.N2 (VSSQ_2), IC2.N5 (VSSQ_3), IC2.P4 (VSSQ_4), IC2.P6 (VSSQ_5), J3.6 (VSS)
- net MMC_CLK: now also J3.5 (CLK), RN2.1 (R1.1)
- net MMC_CMD: now also J3.3 (CMD), RN2.2 (R2.1)
- net MMC_DAT0: now also J3.7 (DAT0), RN2.3 (R3.1)
- net MMC_DAT1: now also J3.8 (DAT1), RN2.4 (R4.1)
- net MMC_DAT2: now also J3.1 (DAT2), RN2.5 (R5.1)
- net MMC_DAT3: now also J3.2 (DAT3/CD), RN2.6 (R6.1)
- net at U1.P1 (GPMC_CSN2): now also IC2.M5 (CMD), RN1.2 (R2.1)
- net at U1.P2 (GPMC_CSN1): now also IC2.M6 (CLK), RN1.3 (R3.1)
- net at U1.P4 (GPMC_AD6): now also IC2.B5 (DAT6), RN1.5 (R5.1)
- net at U1.R1 (GPMC_AD2): now also IC2.A5 (DAT2), RN1.9 (R9.1)
- net at U1.R13 (GPMC_A4): now also IC2.K5 (RESET), RN1.1 (R1.1)
- net at U1.R2 (GPMC_AD1): now also IC2.A4 (DAT1), RN1.10 (R10.1)
- net at U1.R3 (GPMC_AD0): now also IC2.A3 (DAT0), RN1.11 (R11.1)
- net at U1.R4 (GPMC_AD7): now also IC2.B6 (DAT7), RN1.4 (R4.1)
- net at U1.T1 (GPMC_AD5): now also IC2.B4 (DAT5), RN1.6 (R6.1)
- net at U1.T2 (GPMC_AD4): now also IC2.B3 (DAT4), RN1.7 (R7.1)
- net at U1.T3 (GPMC_AD3): now also IC2.B2 (DAT3), RN1.8 (R8.1)
- net UART0_RX renamed CAM_RX
- net UART0_TX renamed CAM_TX
- new net: C17.1, IC2.C2 (VDDI)
- new net +3.3V: C18.1, C19.1, C20.1, C21.1, C22.1, IC2.C6 (VCCQ_1), IC2.E6 (VCC_1), IC2.F5 (VCC_2), IC2.J10 (VCC_3), IC2.K9 (VCC_4), IC2.M4 (VCCQ_2), IC2.N4 (VCCQ_3), IC2.P3 (VCCQ_4), IC2.P5 (VCCQ_5), J3.4 (VDD), RN1.12 (R11.2), RN1.13 (R10.2), RN1.14 (R9.2), RN1.15 (R8.2), RN1.16 (R7.2), RN1.17 (R6.2), RN1.18 (R5.2), RN1.19 (R4.2), RN1.20 (R3.2), RN1.21 (R2.2), RN1.22 (R1.2), RN2.10 (R3.2), RN2.11 (R2.2), RN2.12 (R1.2), RN2.7 (R6.2), RN2.8 (R5.2), RN2.9 (R4.2)
- no-connect marks 6 -> 22
Other:
- moved on the sheet: C10, C11, C12, C13, C14, C15, C16, R8, U1B, U1C, Y1, Y2
