File: osd3358_board.kicad_sch (KiCad schematic)
At the start: 0 parts

Commit message: added emmc and sd
Other:
- sheet Debug Connector renamed Connectors
- sheet Connectors: file debug.kicad_sch -> connectors.kicad_sch
Changed lines of the file:
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@@
 			(color 0 0 0 0.0000)
 		)
-		(property "Sheetname" "Debug Connector"
+		(property "Sheetname" "Connectors"
 			(at 25.4 55.1684 0)
 			(effects
@@
 			)
 		)
-		(property "Sheetfile" "debug.kicad_sch"
+		(property "Sheetfile" "connectors.kicad_sch"
 			(at 25.4 64.0846 0)
 			(effects
